File: lmarv-1/register-card/register-card.sch (KiCad schematic (older format))
At the start: 101 parts, among them P1 dual-pcie-cardedge, P2 CONN_01X02, P3 CONN_01X02, U1 74LVTH16374, U2 74LVTH162541, U3 74LVTH162541, U4 74LVTH16374, U5 74LVTH162541, U6 74LVTH162541

Commit message: Updated register card and breakout
Parts:
- removed U2, U3, U5, U6: 74LVTH162541, Housings_SSOP:SSOP-48_7.5x15.9mm_Pitch0.635mm, symbol 74LVTH162541
- added R35: 1k5, Resistors_SMD:R_0603, symbol R
- added U2, U3, U5, U6: 74LVT16374, Housings_SSOP:SSOP-48_7.5x15.9mm_Pitch0.635mm, symbol 74LVTH16374
- P2, P3: footprint Pin_Headers:Pin_Header_Straight_1x02_Pitch2.54mm -> Pin_Headers:Pin_Header_Straight_1x02_Pitch1.27mm
- U1, U4: value 74LVTH16374 -> 74LVT16374
Connections:
- net GNDREF: now also D1.1 (K), D10.1 (K), D11.1 (K), D12.1 (K), D13.1 (K), D14.1 (K), D15.1 (K), D16.1 (K), D17.1 (K), D18.1 (K), D19.1 (K), D2.1 (K), D20.1 (K), D21.1 (K), D22.1 (K), D23.1 (K), D24.1 (K), D25.1 (K), D26.1 (K), D27.1 (K), D28.1 (K), D29.1 (K), D3.1 (K), D30.1 (K), D31.1 (K), D32.1 (K), D4.1 (K), D5.1 (K), D6.1 (K), D7.1 (K), D8.1 (K), D9.1 (K), U2.10 (GND), U2.15 (GND), U2.21 (GND), U2.28 (GND), U2.34 (GND), U2.39 (GND), U2.4 (GND), U2.45 (GND), U3.10 (GND), U3.15 (GND), U3.21 (GND), U3.28 (GND), U3.34 (GND), U3.39 (GND), U3.4 (GND), U3.45 (GND), U5.10 (GND), U5.15 (GND), U5.21 (GND), U5.28 (GND), U5.34 (GND), U5.39 (GND), U5.4 (GND), U5.45 (GND), U6.10 (GND), U6.15 (GND), U6.21 (GND), U6.28 (GND), U6.34 (GND), U6.39 (GND), U6.4 (GND), U6.45 (GND); no longer U1.1 (1~OE), U1.24 (2~OE), U4.1 (1~OE), U4.24 (2~OE)
- net VDD: now also R35.1, U2.18 (VCC), U2.31 (VCC), U2.42 (VCC), U2.7 (VCC), U3.18 (VCC), U3.31 (VCC), U3.42 (VCC), U3.7 (VCC), U5.18 (VCC), U5.31 (VCC), U5.42 (VCC), U5.7 (VCC), U6.18 (VCC), U6.31 (VCC), U6.42 (VCC), U6.7 (VCC)
- net rd[0]: now also U5.47 (1D1), U6.47 (1D1)
- net rd[10]: now also U5.33 (2D3), U6.33 (2D3)
- net rd[11]: now also U5.32 (2D4), U6.32 (2D4)
- net rd[12]: now also U5.30 (2D5), U6.30 (2D5)
- net rd[13]: now also U5.29 (2D6), U6.29 (2D6)
- net rd[14]: now also U5.27 (2D7), U6.27 (2D7)
- net rd[15]: now also U5.26 (2D8), U6.26 (2D8)
- net rd[16]: now also U2.47 (1D1), U3.47 (1D1)
- net rd[17]: now also U2.46 (1D2), U3.46 (1D2)
- net rd[18]: now also U2.44 (1D3), U3.44 (1D3)
- net rd[19]: now also U2.43 (1D4), U3.43 (1D4)
- net rd[1]: now also U5.46 (1D2), U6.46 (1D2)
- net rd[20]: now also U2.41 (1D5), U3.41 (1D5)
- net rd[21]: now also U2.40 (1D6), U3.40 (1D6)
- net rd[22]: now also U2.38 (1D7), U3.38 (1D7)
- net rd[23]: now also U2.37 (1D8), U3.37 (1D8)
- net rd[24]: now also U2.36 (2D1), U3.36 (2D1)
- net rd[25]: now also U2.35 (2D2), U3.35 (2D2)
- net rd[26]: now also U2.33 (2D3), U3.33 (2D3)
- net rd[27]: now also U2.32 (2D4), U3.32 (2D4)
- net rd[28]: now also U2.30 (2D5), U3.30 (2D5)
- net rd[29]: now also U2.29 (2D6), U3.29 (2D6)
- net rd[2]: now also U5.44 (1D3), U6.44 (1D3)
- net rd[30]: now also U2.27 (2D7), U3.27 (2D7)
- net rd[31]: now also U2.26 (2D8), U3.26 (2D8)
- net rd[3]: now also U5.43 (1D4), U6.43 (1D4)
- net rd[4]: now also U5.41 (1D5), U6.41 (1D5)
- net rd[5]: now also U5.40 (1D6), U6.40 (1D6)
- net rd[6]: now also U5.38 (1D7), U6.38 (1D7)
- net rd[7]: now also U5.37 (1D8), U6.37 (1D8)
- net rd[8]: now also U5.36 (2D1), U6.36 (2D1)
- net rd[9]: now also U5.35 (2D2), U6.35 (2D2)
- net rdclk: now also U2.25 (2CLK), U2.48 (1CLK), U3.25 (2CLK), U3.48 (1CLK), U5.25 (2CLK), U5.48 (1CLK), U6.25 (2CLK), U6.48 (1CLK)
- net rdq[0]: now also U6.2 (1Q1); no longer U4.2 (1Q1)
- net rdq[10]: now also U6.16 (2Q3); no longer U4.16 (2Q3)
- net rdq[11]: now also U6.17 (2Q4); no longer U4.17 (2Q4)
- net rdq[12]: now also U6.19 (2Q5); no longer U4.19 (2Q5)
- net rdq[13]: now also U6.20 (2Q6); no longer U4.20 (2Q6)
- net rdq[14]: now also U6.22 (2Q7); no longer U4.22 (2Q7)
- net rdq[15]: now also U6.23 (2Q8); no longer U4.23 (2Q8)
- net rdq[16]: now also U3.2 (1Q1); no longer U1.2 (1Q1)
- net rdq[17]: now also U3.3 (1Q2); no longer U1.3 (1Q2)
- net rdq[18]: now also U3.5 (1Q3); no longer U1.5 (1Q3)
- net rdq[19]: now also U3.6 (1Q4); no longer U1.6 (1Q4)
- net rdq[1]: now also U6.3 (1Q2); no longer U4.3 (1Q2)
- net rdq[20]: now also U3.8 (1Q5); no longer U1.8 (1Q5)
- net rdq[21]: now also U3.9 (1Q6); no longer U1.9 (1Q6)
- net rdq[22]: now also U3.11 (1Q7); no longer U1.11 (1Q7)
- net rdq[23]: now also U3.12 (1Q8); no longer U1.12 (1Q8)
- net rdq[24]: now also U3.13 (2Q1); no longer U1.13 (2Q1)
- net rdq[25]: now also U3.14 (2Q2); no longer U1.14 (2Q2)
- net rdq[26]: now also U3.16 (2Q3); no longer U1.16 (2Q3)
- net rdq[27]: now also U3.17 (2Q4); no longer U1.17 (2Q4)
- net rdq[28]: now also U3.19 (2Q5); no longer U1.19 (2Q5)
- net rdq[29]: now also U3.20 (2Q6); no longer U1.20 (2Q6)
- net rdq[2]: now also U6.5 (1Q3); no longer U4.5 (1Q3)
- net rdq[30]: now also U3.22 (2Q7); no longer U1.22 (2Q7)
- net rdq[31]: now also U3.23 (2Q8); no longer U1.23 (2Q8)
- net rdq[3]: now also U6.6 (1Q4); no longer U4.6 (1Q4)
- net rdq[4]: now also U6.8 (1Q5); no longer U4.8 (1Q5)
- net rdq[5]: now also U6.9 (1Q6); no longer U4.9 (1Q6)
- net rdq[6]: now also U6.11 (1Q7); no longer U4.11 (1Q7)
- net rdq[7]: now also U6.12 (1Q8); no longer U4.12 (1Q8)
- net rdq[8]: now also U6.13 (2Q1); no longer U4.13 (2Q1)
- net rdq[9]: now also U6.14 (2Q2); no longer U4.14 (2Q2)
- net rs1[0]: now also U4.2 (1Q1)
- net rs1[10]: now also U4.16 (2Q3)
- net rs1[11]: now also U4.17 (2Q4)
- net rs1[12]: now also U4.19 (2Q5)
- net rs1[13]: now also U4.20 (2Q6)
- net rs1[14]: now also U4.22 (2Q7)
- net rs1[15]: now also U4.23 (2Q8)
- net rs1[16]: now also U1.2 (1Q1)
- net rs1[17]: now also U1.3 (1Q2)
- net rs1[18]: now also U1.5 (1Q3)
- net rs1[19]: now also U1.6 (1Q4)
- net rs1[1]: now also U4.3 (1Q2)
- net rs1[20]: now also U1.8 (1Q5)
- net rs1[21]: now also U1.9 (1Q6)
- net rs1[22]: now also U1.11 (1Q7)
- net rs1[23]: now also U1.12 (1Q8)
- net rs1[24]: now also U1.13 (2Q1)
- net rs1[25]: now also U1.14 (2Q2)
- net rs1[26]: now also U1.16 (2Q3)
- net rs1[27]: now also U1.17 (2Q4)
- net rs1[28]: now also U1.19 (2Q5)
- net rs1[29]: now also U1.20 (2Q6)
- net rs1[2]: now also U4.5 (1Q3)
- net rs1[30]: now also U1.22 (2Q7)
- net rs1[31]: now also U1.23 (2Q8)
- net rs1[3]: now also U4.6 (1Q4)
- net rs1[4]: now also U4.8 (1Q5)
- net rs1[5]: now also U4.9 (1Q6)
- net rs1[6]: now also U4.11 (1Q7)
- net rs1[7]: now also U4.12 (1Q8)
- net rs1[8]: now also U4.13 (2Q1)
- net rs1[9]: now also U4.14 (2Q2)
- net rs2[0]: now also U5.2 (1Q1)
- net rs2[10]: now also U5.16 (2Q3)
- net rs2[11]: now also U5.17 (2Q4)
- net rs2[12]: now also U5.19 (2Q5)
- net rs2[13]: now also U5.20 (2Q6)
- net rs2[14]: now also U5.22 (2Q7)
- net rs2[15]: now also U5.23 (2Q8)
- net rs2[16]: now also U2.2 (1Q1)
- net rs2[17]: now also U2.3 (1Q2)
- net rs2[18]: now also U2.5 (1Q3)
- net rs2[19]: now also U2.6 (1Q4)
- net rs2[1]: now also U5.3 (1Q2)
- net rs2[20]: now also U2.8 (1Q5)
- net rs2[21]: now also U2.9 (1Q6)
- net rs2[22]: now also U2.11 (1Q7)
- net rs2[23]: now also U2.12 (1Q8)
- net rs2[24]: now also U2.13 (2Q1)
- net rs2[25]: now also U2.14 (2Q2)
- net rs2[26]: now also U2.16 (2Q3)
- net rs2[27]: now also U2.17 (2Q4)
- net rs2[28]: now also U2.19 (2Q5)
- net rs2[29]: now also U2.20 (2Q6)
- net rs2[2]: now also U5.5 (1Q3)
- net rs2[30]: now also U2.22 (2Q7)
- net rs2[31]: now also U2.23 (2Q8)
- net rs2[3]: now also U5.6 (1Q4)
- net rs2[4]: now also U5.8 (1Q5)
- net rs2[5]: now also U5.9 (1Q6)
- net rs2[6]: now also U5.11 (1Q7)
- net rs2[7]: now also U5.12 (1Q8)
- net rs2[8]: now also U5.13 (2Q1)
- net rs2[9]: now also U5.14 (2Q2)
- net ~rs1oe: now also U1.1 (1~OE), U1.24 (2~OE), U4.1 (1~OE), U4.24 (2~OE)
- net ~rs2oe: now also U2.1 (1~OE), U2.24 (2~OE), U5.1 (1~OE), U5.24 (2~OE)
- new net: P2.2 (P2), R35.2, U3.1 (1~OE), U3.24 (2~OE), U6.1 (1~OE), U6.24 (2~OE)
Other:
- note added: "DISPLAY STORAGE"
- note added: "REGISTER CONTENT INDICATORS"
- note added: "REGISTER CONTENT\nINDICATOR ENABLE"
- note added: "SOURCE 1 STORAGE"
- note added: "SOURCE 2 STORAGE"
- note added: "rs1oe INDICATOR"
- note added: "rs2oe INDICATOR"
- note added: "rsoe INDICATOR ENABLE"
- moved on the sheet: D1, D10, D11, D12, D13, D14, D15, D16, D17, D18, D19, D2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

Commit message: Adds RAM-based register card
Parts:
- added C71, C72, C73, C74, C81, C82, C83, C84: 100n, Capacitors_SMD:C_0603, symbol Device:C
- added U7, U8: 74LVT162244, Housings_SSOP:SSOP-48_7.5x15.9mm_Pitch0.635mm, symbol lmarv:74LVTH162541
- C11: renamed from C1; symbol C -> Device:C
- C12: renamed from C2; symbol C -> Device:C
- C13: renamed from C3; symbol C -> Device:C
- C14: renamed from C4; symbol C -> Device:C
- C21: renamed from C13; symbol C -> Device:C
- C22: renamed from C14; symbol C -> Device:C
- C23: renamed from C15; symbol C -> Device:C
- C24: renamed from C16; symbol C -> Device:C
- C31: renamed from C5; symbol C -> Device:C
- C32: renamed from C6; symbol C -> Device:C
- C33: renamed from C7; symbol C -> Device:C
- C34: renamed from C8; symbol C -> Device:C
- C41: renamed from C17; symbol C -> Device:C
- C42: renamed from C18; symbol C -> Device:C
- C43: renamed from C19; symbol C -> Device:C
- C44: renamed from C20; symbol C -> Device:C
- C51: renamed from C9; symbol C -> Device:C
- C52: renamed from C10; symbol C -> Device:C
- C53: renamed from C11; symbol C -> Device:C
- C54: renamed from C12; symbol C -> Device:C
- C61: renamed from C21; symbol C -> Device:C
- C62: renamed from C22; symbol C -> Device:C
- C63: renamed from C23; symbol C -> Device:C
- C64: renamed from C24; symbol C -> Device:C
- D1, D10, D11, D12, D13, D14, D15, D16, D17, D18, D19, D2, D20, D21, D22, D23, D24, D25, D26, D27, D28, D29, D3, D30, D31, D32, D33, D34, D4, D5, D6, D7, D8, D9: symbol LED -> register-card-rescue:LED-RESCUE-register-card
- P1: symbol dual-pcie-cardedge -> lmarv:dual-pcie-cardedge
- P2, P3: symbol CONN_01X02 -> register-card-rescue:CONN_01X02-RESCUE-register-card
- R1, R10, R11, R12, R13, R14, R15, R16, R17, R18, R19, R2, R20, R21, R22, R23, R24, R25, R26, R27, R28, R29, R3, R30, R31, R32, R33, R34, R35, R4, R5, R6, R7, R8, R9: symbol R -> Device:R
- U1, U2, U3, U4, U5, U6: symbol 74LVTH16374 -> lmarv:74LVTH16374
Connections:
- net GNDREF: now also C71.2, C72.2, C73.2, C74.2, C81.2, C82.2, C83.2, C84.2, U7.1 (1~OE1), U7.10 (GND), U7.15 (GND), U7.21 (GND), U7.24 (2~OE1), U7.25 (2~OE2), U7.28 (GND), U7.34 (GND), U7.39 (GND), U7.4 (GND), U7.45 (GND), U7.48 (1~OE2), U8.1 (1~OE1), U8.10 (GND), U8.15 (GND), U8.21 (GND), U8.24 (2~OE1), U8.25 (2~OE2), U8.28 (GND), U8.34 (GND), U8.39 (GND), U8.4 (GND), U8.45 (GND), U8.48 (1~OE2)
- net VDD: now also C71.1, C72.1, C73.1, C74.1, C81.1, C82.1, C83.1, C84.1, U7.18 (VCC), U7.31 (VCC), U7.42 (VCC), U7.7 (VCC), U8.18 (VCC), U8.31 (VCC), U8.42 (VCC), U8.7 (VCC)
- net rd[0]: now also U8.47 (1A1); no longer U4.47 (1D1), U5.47 (1D1), U6.47 (1D1)
- net rd[10]: now also U8.33 (2A3); no longer U4.33 (2D3), U5.33 (2D3), U6.33 (2D3)
- net rd[11]: now also U8.32 (2A4); no longer U4.32 (2D4), U5.32 (2D4), U6.32 (2D4)
- net rd[12]: now also U8.30 (2A5); no longer U4.30 (2D5), U5.30 (2D5), U6.30 (2D5)
- net rd[13]: now also U8.29 (2A6); no longer U4.29 (2D6), U5.29 (2D6), U6.29 (2D6)
- net rd[14]: now also U8.27 (2A7); no longer U4.27 (2D7), U5.27 (2D7), U6.27 (2D7)
- net rd[15]: now also U8.26 (2A8); no longer U4.26 (2D8), U5.26 (2D8), U6.26 (2D8)
- net rd[16]: now also U7.47 (1A1); no longer U1.47 (1D1), U2.47 (1D1), U3.47 (1D1)
- net rd[17]: now also U7.46 (1A2); no longer U1.46 (1D2), U2.46 (1D2), U3.46 (1D2)
- net rd[18]: now also U7.44 (1A3); no longer U1.44 (1D3), U2.44 (1D3), U3.44 (1D3)
- net rd[19]: now also U7.43 (1A4); no longer U1.43 (1D4), U2.43 (1D4), U3.43 (1D4)
- net rd[1]: now also U8.46 (1A2); no longer U4.46 (1D2), U5.46 (1D2), U6.46 (1D2)
- net rd[20]: now also U7.41 (1A5); no longer U1.41 (1D5), U2.41 (1D5), U3.41 (1D5)
- net rd[21]: now also U7.40 (1A6); no longer U1.40 (1D6), U2.40 (1D6), U3.40 (1D6)
- net rd[22]: now also U7.38 (1A7); no longer U1.38 (1D7), U2.38 (1D7), U3.38 (1D7)
- net rd[23]: now also U7.37 (1A8); no longer U1.37 (1D8), U2.37 (1D8), U3.37 (1D8)
- net rd[24]: now also U7.36 (2A1); no longer U1.36 (2D1), U2.36 (2D1), U3.36 (2D1)
- net rd[25]: now also U7.35 (2A2); no longer U1.35 (2D2), U2.35 (2D2), U3.35 (2D2)
- net rd[26]: now also U7.33 (2A3); no longer U1.33 (2D3), U2.33 (2D3), U3.33 (2D3)
- net rd[27]: now also U7.32 (2A4); no longer U1.32 (2D4), U2.32 (2D4), U3.32 (2D4)
- net rd[28]: now also U7.30 (2A5); no longer U1.30 (2D5), U2.30 (2D5), U3.30 (2D5)
- net rd[29]: now also U7.29 (2A6); no longer U1.29 (2D6), U2.29 (2D6), U3.29 (2D6)
- net rd[2]: now also U8.44 (1A3); no longer U4.44 (1D3), U5.44 (1D3), U6.44 (1D3)
- net rd[30]: now also U7.27 (2A7); no longer U1.27 (2D7), U2.27 (2D7), U3.27 (2D7)
- net rd[31]: now also U7.26 (2A8); no longer U1.26 (2D8), U2.26 (2D8), U3.26 (2D8)
- net rd[3]: now also U8.43 (1A4); no longer U4.43 (1D4), U5.43 (1D4), U6.43 (1D4)
- net rd[4]: now also U8.41 (1A5); no longer U4.41 (1D5), U5.41 (1D5), U6.41 (1D5)
- net rd[5]: now also U8.40 (1A6); no longer U4.40 (1D6), U5.40 (1D6), U6.40 (1D6)
- net rd[6]: now also U8.38 (1A7); no longer U4.38 (1D7), U5.38 (1D7), U6.38 (1D7)
- net rd[7]: now also U8.37 (1A8); no longer U4.37 (1D8), U5.37 (1D8), U6.37 (1D8)
- net rd[8]: now also U8.36 (2A1); no longer U4.36 (2D1), U5.36 (2D1), U6.36 (2D1)
- net rd[9]: now also U8.35 (2A2); no longer U4.35 (2D2), U5.35 (2D2), U6.35 (2D2)
- net /LEDOE: now reaches P2.2 (P2), R35.2, U3.1 (1~OE), U3.24 (2~OE), U6.1 (1~OE), U6.24 (2~OE)
- new net dd[0]: U4.47 (1D1), U5.47 (1D1), U6.47 (1D1), U8.2 (1Y1)
- new net dd[10]: U4.33 (2D3), U5.33 (2D3), U6.33 (2D3), U8.16 (2Y3)
- new net dd[11]: U4.32 (2D4), U5.32 (2D4), U6.32 (2D4), U8.17 (2Y4)
- new net dd[12]: U4.30 (2D5), U5.30 (2D5), U6.30 (2D5), U8.19 (2Y5)
- new net dd[13]: U4.29 (2D6), U5.29 (2D6), U6.29 (2D6), U8.20 (2Y6)
- new net dd[14]: U4.27 (2D7), U5.27 (2D7), U6.27 (2D7), U8.22 (2Y7)
- new net dd[15]: U4.26 (2D8), U5.26 (2D8), U6.26 (2D8), U8.23 (2Y8)
- new net dd[16]: U1.47 (1D1), U2.47 (1D1), U3.47 (1D1), U7.2 (1Y1)
- new net dd[17]: U1.46 (1D2), U2.46 (1D2), U3.46 (1D2), U7.3 (1Y2)
- new net dd[18]: U1.44 (1D3), U2.44 (1D3), U3.44 (1D3), U7.5 (1Y3)
- new net dd[19]: U1.43 (1D4), U2.43 (1D4), U3.43 (1D4), U7.6 (1Y4)
- new net dd[1]: U4.46 (1D2), U5.46 (1D2), U6.46 (1D2), U8.3 (1Y2)
- new net dd[20]: U1.41 (1D5), U2.41 (1D5), U3.41 (1D5), U7.8 (1Y5)
- new net dd[21]: U1.40 (1D6), U2.40 (1D6), U3.40 (1D6), U7.9 (1Y6)
- new net dd[22]: U1.38 (1D7), U2.38 (1D7), U3.38 (1D7), U7.11 (1Y7)
- new net dd[23]: U1.37 (1D8), U2.37 (1D8), U3.37 (1D8), U7.12 (1Y8)
- new net dd[24]: U1.36 (2D1), U2.36 (2D1), U3.36 (2D1), U7.13 (2Y1)
- new net dd[25]: U1.35 (2D2), U2.35 (2D2), U3.35 (2D2), U7.14 (2Y2)
- new net dd[26]: U1.33 (2D3), U2.33 (2D3), U3.33 (2D3), U7.16 (2Y3)
- new net dd[27]: U1.32 (2D4), U2.32 (2D4), U3.32 (2D4), U7.17 (2Y4)
- new net dd[28]: U1.30 (2D5), U2.30 (2D5), U3.30 (2D5), U7.19 (2Y5)
- new net dd[29]: U1.29 (2D6), U2.29 (2D6), U3.29 (2D6), U7.20 (2Y6)
- new net dd[2]: U4.44 (1D3), U5.44 (1D3), U6.44 (1D3), U8.5 (1Y3)
- new net dd[30]: U1.27 (2D7), U2.27 (2D7), U3.27 (2D7), U7.22 (2Y7)
- new net dd[31]: U1.26 (2D8), U2.26 (2D8), U3.26 (2D8), U7.23 (2Y8)
- new net dd[3]: U4.43 (1D4), U5.43 (1D4), U6.43 (1D4), U8.6 (1Y4)
- new net dd[4]: U4.41 (1D5), U5.41 (1D5), U6.41 (1D5), U8.8 (1Y5)
- new net dd[5]: U4.40 (1D6), U5.40 (1D6), U6.40 (1D6), U8.9 (1Y6)
- new net dd[6]: U4.38 (1D7), U5.38 (1D7), U6.38 (1D7), U8.11 (1Y7)
- new net dd[7]: U4.37 (1D8), U5.37 (1D8), U6.37 (1D8), U8.12 (1Y8)
- new net dd[8]: U4.36 (2D1), U5.36 (2D1), U6.36 (2D1), U8.13 (2Y1)
- new net dd[9]: U4.35 (2D2), U5.35 (2D2), U6.35 (2D2), U8.14 (2Y2)
Other:
- note added: "CARD INPUT BUFFER"
- moved on the sheet: C11, C12, C13, C14, C21, C22, C23, C24, C31, C32, C33, C34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
