File: card-breakout/card-breakout.sch (KiCad schematic (older format))
At the start: 11 parts, among them P1 CONN_01X05, P10 CONN_01X05, P11 CONN_01X05, P2 CONN_01X05, P3 CONN_01X32, P4 CONN_01X32, P5 dual-pcie-cardedge, P6 CONN_02X01, P7 CONN_01X32, P8 CONN_01X32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

Commit message: Dump for backing up, 2018 Jul 7
Parts:
- P1, P10, P11, P2: symbol CONN_01X05 -> card-breakout-rescue:CONN_01X05
- P3, P4, P7, P8: symbol CONN_01X32 -> card-breakout-rescue:CONN_01X32
- P5: symbol dual-pcie-cardedge -> lmarv1:dual-pcie-cardedge
- P6, P9: symbol CONN_02X01 -> card-breakout-rescue:CONN_02X01
Changed lines of the file:
@@
-EESchema Schematic File Version 2
-LIBS:power
-LIBS:device
-LIBS:transistors
-LIBS:conn
-LIBS:linear
-LIBS:regul
-LIBS:74xx
-LIBS:cmos4000
-LIBS:adc-dac
-LIBS:memory
-LIBS:xilinx
-LIBS:microcontrollers
-LIBS:dsp
-LIBS:microchip
-LIBS:analog_switches
-LIBS:motorola
-LIBS:texas
-LIBS:intel
-LIBS:audio
-LIBS:interface
-LIBS:digital-audio
-LIBS:philips
-LIBS:display
-LIBS:cypress
-LIBS:siliconi
-LIBS:opto
-LIBS:atmel
-LIBS:contrib
-LIBS:valves
-LIBS:lmarv
-EELAYER 25 0
+EESchema Schematic File Version 4
+LIBS:card-breakout-cache
+EELAYER 26 0
 EELAYER END
 $Descr A4 11693 8268
@@
 $EndDescr
 $Comp
-L dual-pcie-cardedge P5
+L lmarv1:dual-pcie-cardedge P5
 U 1 1 5A71167D
 P 5950 3800
@@
 $EndComp
 $Comp
-L CONN_02X01 P6
+L card-breakout-rescue:CONN_02X01 P6
 U 1 1 5A7119A6
 P 10325 5125
@@
 $EndComp
 $Comp
-L CONN_02X01 P9
+L card-breakout-rescue:CONN_02X01 P9
 U 1 1 5A711A53
 P 1575 5550
@@
 	9750 4400 9750 5300
 $Comp
-L CONN_01X32 P8
+L card-breakout-rescue:CONN_01X32 P8
 U 1 1 5A711E6D
 P 8200 5500
@@
 $EndComp
 $Comp
-L CONN_01X32 P7
+L card-breakout-rescue:CONN_01X32 P7
 U 1 1 5A711F7E
 P 4200 5500
@@
 	9750 3200 9750 2300
 $Comp
-L CONN_01X32 P4
+L card-breakout-rescue:CONN_01X32 P4
 U 1 1 5A712206
 P 8200 2100
@@
 	5750 3200 5750 2300
 $Comp
-L CONN_01X32 P3
+L card-breakout-rescue:CONN_01X32 P3
 U 1 1 5A712340
 P 4200 2100
@@
 $EndComp
 $Comp
-L CONN_01X05 P11
+L card-breakout-rescue:CONN_01X05 P11
 U 1 1 5A7123C1
 P 6350 5825
@@
 	6150 4400 6150 5625
 $Comp
-L CONN_01X05 P10
+L card-breakout-rescue:CONN_01X05 P10
 U 1 1 5A7126C6
 P 2350 5825
@@
 	2150 4400 2150 5625
 $Comp
-L CONN_01X05 P1
+L card-breakout-rescue:CONN_01X05 P1
 U 1 1 5A712893
 P 2350 1775
@@
 	1575 5300 1575 3800
 Wire Wire Line
-	1575 3800 1850 3800
+	1575 3800 1825 3800
 Wire Wire Line
 	1575 5800 1825 5800
@@
 Connection ~ 1825 3800
 Wire Wire Line
-	10050 3800 10325 3800
+	10050 3800 10100 3800
 Wire Wire Line
 	10325 3800 10325 4875
@@
 Connection ~ 10100 3800
 $Comp
-L CONN_01X05 P2
+L card-breakout-rescue:CONN_01X05 P2
 U 1 1 5A7135FB
 P 6350 1775
@@
 Text Label 10325 4550 1    60   ~ 0
 VDD
+Wire Wire Line
+	1825 3800 1850 3800
+Wire Wire Line
+	10100 3800 10325 3800
 $EndSCHEMATC
