File: lmarv-1/register-motherboard/register-motherboard.sch (KiCad schematic (older format))
At the start: 143 parts, among them U5 74LVC138, U6 74LVC138, U7 74LVC138

Commit message: Dump for backing up, 2018 Jul 7
Parts:
- removed C?: 160p, symbol Device:C
- removed CN? (x31): CKCA43C0G1H151K, symbol lmarv:CKCA43C0G1H
- removed PR1, PR2, PR? (x30): dual-pcie-cardedge, lmarv:2pci_express_slot, symbol lmarv:dual-pcie-cardedge
- removed R?: 100R, symbol Device:R
- removed RN? (x31): CAT16-101J4, symbol Device:R_Pack04
- removed U5, U6, U7, U? (x9): 74LVC138, Housings_SOIC:SOIC-16_3.9x9.9mm_Pitch1.27mm, symbol register-motherboard-rescue:74LS138-RESCUE-register-motherboard
- removed U? (x32): 74LVC1G02, symbol Logic_74xgxx:74LVC1G02
- removed U?: 74LVC04, symbol lmarv:74LVC04
- added C1, C10, C11, C12, C13, C14, C2, C3, C4, C5, C6, C7, C8, C9: 47u, Capacitors_SMD:CP_Elec_4x4.5, symbol Device:CP
- added CN10, CN11, CN12, CN13, CN14, CN15, CN16, CN17, CN18, CN19, CN2, CN20, CN21, CN22, CN23, CN24, CN25, CN26, CN27, CN28, CN29, CN3, CN30, CN31, CN32, CN33, CN34, CN35, CN36, CN37, CN38, CN39, CN4, CN40, CN41, CN42, CN43, CN44, CN45, CN46, CN47, CN48, CN49, CN5, CN50, CN51, CN52, CN53, CN54, CN55, CN56, CN57, CN58, CN59, CN6, CN60, CN61, CN62, CN63, CN64, CN65, CN66, CN67, CN68, CN69, CN7, CN70, CN71, CN72, CN73, CN74, CN75, CN76, CN8, CN9: CA0612KRNPO9BN151, lmarv:CARRAY_8_0612_3.2x1.6mm_Pitch0.8mm, symbol lmarv:CKCA43C0G1H
- added P1, P10, P11, P12, P2, P3, P4, P5, P6, P7, P8, P9: dual-pcie-cardedge, lmarv:2pci_express_slot, symbol lmarv:dual-pcie-cardedge
- added RN10, RN11, RN12, RN13, RN14, RN15, RN16, RN17, RN18, RN19, RN2, RN20, RN21, RN22, RN23, RN24, RN25, RN26, RN27, RN28, RN29, RN3, RN30, RN31, RN32, RN33, RN34, RN35, RN36, RN37, RN38, RN39, RN4, RN40, RN41, RN42, RN43, RN44, RN45, RN46, RN47, RN48, RN49, RN5, RN50, RN51, RN52, RN53, RN54, RN55, RN56, RN57, RN58, RN59, RN6, RN60, RN61, RN62, RN63, RN64, RN65, RN66, RN67, RN68, RN69, RN7, RN70, RN71, RN72, RN73, RN74, RN75, RN76, RN8, RN9: CAT16-101J4, lmarv:CARRAY_8_0612_3.2x1.6mm_Pitch0.8mm, symbol Device:R_Pack04
- CN1: renamed from CN?; value CKCA43C0G1H151K -> CA0612KRNPO9BN151; footprint (none) -> lmarv:CARRAY_8_0612_3.2x1.6mm_Pitch0.8mm; MFG (none) -> Yageo; MFG P/N (none) -> CA0612KRNPO9BN151
- RN1: renamed from RN?; footprint (none) -> lmarv:CARRAY_8_0612_3.2x1.6mm_Pitch0.8mm; MFG (none) -> Bourns; MFG P/N (none) -> CAT16-101J4
Connections:
- net labels added: BOOT_CLK, GND, VDD, f[0], f[1], f[2], f[3], nc0, nc1, nc10, nc11, nc12, nc2, nc3, nc4, nc5, nc6, nc7, nc8, nc9, rda[0], rda[1], rda[2], rda[3], rda[4], rs1a[0], rs1a[1], rs1a[2], rs1a[3], rs1a[4], rs2a[0], rs2a[1], rs2a[2], rs2a[3], rs2a[4], ~BOOT_ALU_EN, ~BOOT_RST, ~BOOT_WR, ~alu_oe, ~rd_bhh, ~rd_bhl, ~rd_blh, ~rd_bll, ~rd_wr, ~rs1_bhh, ~rs1_bhl, ~rs1_blh, ~rs1_bll, ~rs1_rd, ~rs2_bhh, ~rs2_bhl, ~rs2_blh, ~rs2_bll, ~rs2_rd
- net labels removed: RDCLK[0], RDCLK[10], RDCLK[11], RDCLK[12], RDCLK[13], RDCLK[14], RDCLK[15], RDCLK[16], RDCLK[17], RDCLK[18], RDCLK[19], RDCLK[1], RDCLK[20], RDCLK[22], RDCLK[23], RDCLK[24], RDCLK[25], RDCLK[26], RDCLK[27], RDCLK[28], RDCLK[29], RDCLK[2], RDCLK[30], RDCLK[31], RDCLK[3], RDCLK[4], RDCLK[5], RDCLK[6], RDCLK[7], RDCLK[8], RDCLK[9], rdsel[0], rdsel[1], rdsel[2], rdsel[3], rdsel[4], rs1sel[0], rs1sel[1], rs1sel[2], rs1sel[3], rs1sel[4], rs2sel[0], rs2sel[1], rs2sel[2], rs2sel[3], rs2sel[4], ~RDCLK, ~RDCLKEN[0], ~RDCLKEN[10], ~RDCLKEN[11], ~RDCLKEN[12], ~RDCLKEN[13], ~RDCLKEN[14], ~RDCLKEN[15], ~RDCLKEN[16], ~RDCLKEN[17], ~RDCLKEN[18], ~RDCLKEN[19], ~RDCLKEN[1], ~RDCLKEN[20], ~RDCLKEN[21], ~RDCLKEN[22], ~RDCLKEN[23], ~RDCLKEN[24], ~RDCLKEN[25], ~RDCLKEN[26], ~RDCLKEN[27], ~RDCLKEN[28], ~RDCLKEN[29], ~RDCLKEN[2], ~RDCLKEN[30], ~RDCLKEN[31], ~RDCLKEN[3], ~RDCLKEN[4], ~RDCLKEN[5], ~RDCLKEN[6], ~RDCLKEN[7], ~RDCLKEN[8], ~RDCLKEN[9], ~RS1OE[0], ~RS1OE[10], ~RS1OE[11], ~RS1OE[12], ~RS1OE[13], ~RS1OE[14], ~RS1OE[15], ~RS1OE[16], ~RS1OE[17], ~RS1OE[18], ~RS1OE[19], ~RS1OE[1], ~RS1OE[20], ~RS1OE[21], ~RS1OE[22], ~RS1OE[23], ~RS1OE[24], ~RS1OE[25], ~RS1OE[26], ~RS1OE[27], ~RS1OE[28], ~RS1OE[29], ~RS1OE[2], ~RS1OE[30], ~RS1OE[31], ~RS1OE[3], ~RS1OE[4], ~RS1OE[5], ~RS1OE[6], ~RS1OE[7], ~RS1OE[8], ~RS1OE[9], ~RS2OE[0], ~RS2OE[10], ~RS2OE[11], ~RS2OE[12], ~RS2OE[13], ~RS2OE[14], ~RS2OE[15], ~RS2OE[16], ~RS2OE[17], ~RS2OE[18], ~RS2OE[19], ~RS2OE[1], ~RS2OE[20], ~RS2OE[21], ~RS2OE[22], ~RS2OE[23], ~RS2OE[24], ~RS2OE[25], ~RS2OE[26], ~RS2OE[27], ~RS2OE[28], ~RS2OE[29], ~RS2OE[2], ~RS2OE[30], ~RS2OE[31], ~RS2OE[3], ~RS2OE[4], ~RS2OE[5], ~RS2OE[6], ~RS2OE[7], ~RS2OE[8], ~RS2OE[9], ~rdsel[3], ~rs1sel[3], ~rs2sel[3]
- wire segments 3801 -> 2102
- no-connect marks 1569 -> 0
Other:
- note removed: "~RDCLK[0-7]"
- note removed: "~RDCLK[16-23]"
- note removed: "~RDCLK[24-31]"
- note removed: "~RDCLK[8-15]"
- note removed: "~RS1OE[0-7]"
- note removed: "~RS1OE[16-23]"
- note removed: "~RS1OE[24-31]"
- note removed: "~RS1OE[8-15]"
- note removed: "~RS2OE[0-7]"
- note removed: "~RS2OE[16-23]"
- note removed: "~RS2OE[24-31]"
- note removed: "~RS2OE[8-15]"

Commit message: Adds tinyfpga test things
Parts:
- CN1, CN10, CN11, CN12, CN13, CN14, CN15, CN16, CN17, CN18, CN19, CN2, CN20, CN21, CN22, CN23, CN24, CN25, CN26, CN27, CN28, CN29, CN3, CN30, CN31, CN32, CN33, CN34, CN35, CN36, CN37, CN38, CN39, CN4, CN40, CN41, CN42, CN43, CN44, CN45, CN46, CN47, CN48, CN49, CN5, CN50, CN51, CN52, CN53, CN54, CN55, CN56, CN57, CN58, CN59, CN6, CN60, CN61, CN62, CN63, CN64, CN65, CN66, CN67, CN68, CN69, CN7, CN70, CN71, CN72, CN73, CN74, CN75, CN76, CN8, CN9, RN1, RN10, RN11, RN12, RN13, RN14, RN15, RN16, RN17, RN18, RN19, RN2, RN20, RN21, RN22, RN23, RN24, RN25, RN26, RN27, RN28, RN29, RN3, RN30, RN31, RN32, RN33, RN34, RN35, RN36, RN37, RN38, RN39, RN4, RN40, RN41, RN42, RN43, RN44, RN45, RN46, RN47, RN48, RN49, RN5, RN50, RN51, RN52, RN53, RN54, RN55, RN56, RN57, RN58, RN59, RN6, RN60, RN61, RN62, RN63, RN64, RN65, RN66, RN67, RN68, RN69, RN7, RN70, RN71, RN72, RN73, RN74, RN75, RN76, RN8, RN9: footprint lmarv:CARRAY_8_0612_3.2x1.6mm_Pitch0.8mm -> Resistors_SMD:R_Cat16-4
- P1, P10, P11, P12, P2, P3, P4, P5, P6, P7, P8, P9: footprint lmarv:2pci_express_slot -> lmarv:2pci_express_slot_small
Connections:
- no-connect marks 0 -> 4
