File: lmarv-1/shifter/shifter.sch (KiCad schematic (older format))
At the start: 138 parts, among them J1 Conn_02x09_Odd_Even, P1 dual-pcie-cardedge, U1 74LVC541, U10 74LVC541, U11 74LVC541, U12 74LVC541, U13 74LVC541, U14 74LVC541, U15 74LVC541, U16 74LVC541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

Commit message: Adds tinyfpga test things
Parts:
- RN1, RN2: footprint lmarv:YC158 -> lmarv:Yageo_YC358
