File: lmarv-1/tester/tester.sch (KiCad schematic (older format))
At the start: 88 parts, among them P1 dual-pcie-cardedge, U1 74HC597, U10 74HC597, U11 74HC597, U12 74HC597, U13 74LVC595, U14 74LVC595, U15 74LVC595, U16 74LVC595, U17 74HC597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

Commit message: Mainly updates alu.py simulator
Connections:
- wire segments 1118 -> 1102
- no-connect marks 20 -> 19
Other:
- note added: "rs2a[4] GETS\nSHIFTED IN\nFIRST"
- note added: "rs2a[4] GETS\nSHIFTED OUT\nFIRST"
- note removed: "q1 GETS\nSHIFTED IN\nFIRST"
- note removed: "q1 GETS\nSHIFTED OUT\nFIRST"
