File: lmarv-1/alu/alu.sch (KiCad schematic (older format))
At the start: 126 parts, among them J1 Conn_02x03_Odd_Even, J2 Conn_01x01, J3 Conn_01x01, J4 Conn_01x01, P1 dual-pcie-cardedge, Q1 SSM3J358R, Q2 SSM3J358R, Q3 SSM3J358R, U1 74HC590, U10 74LVC541, U11 IS61LV256AL, U12 74LVC541, U13 74LVC541, U14 74LVC541, U15 IS61LV256AL, U16 IS61LV256AL, U17 74LVC541, U18 74LVC541, U19 74LVC541, U2 AT28BV64B-20JU, U20 IS61LV256AL, U21 74LVC541, U22 74LVC541, U23 74LVC541, U24 IS61LV256AL, U25 74LVC541, U26 74LVC541, U27 74LVC541, U28 IS61LV256AL, U29 74LVC541, U3 AT28BV256B-20JU, U30 74LVC541, U31 74LVC541, U32 IS61LV256AL, U33 74LVC541, U34 74LVC541, U35 74LVC541, U36 IS61LV256AL, U37 74LVC541, U38 74LVC541, U39 74LVC541, U4 74HC590, U40 IS61LV256AL, U41 74LVC541, U42 74LVC32, U43 74LVC04, U44 74LVC32, U45 74LVC541, U46 74LVC541, U47 74LVC541, U48 74LVC541, U49 74LVC541, U5 74LVC541, U50 74LVC541, U51 74LVC541, U52 74LVC541, U53 74LVC541, U54 74LVC541, U55 74LVC541, U56 74LVC541, U6 74LVC541, U7 74LVC541, U8 74LVC541, U9 74LVC541

Commit message: Mainly updates alu.py simulator
Parts:
- removed J2, J3, J4: Conn_01x01, Connectors_Samtec:SL-101-X-XX_1x01, symbol Connector_Generic:Conn_01x01
- removed P1: dual-pcie-cardedge, lmarv:PCI-EXPRESS, symbol alu-rescue:dual-pcie-cardedge-lmarv
- removed Q1, Q2, Q3: SSM3J358R, TO_SOT_Packages_SMD:SOT-23_Handsoldering, symbol Device:Q_PMOS_GSD
- removed U1: 74HC590, Housings_SOIC:SOIC-16_3.9x9.9mm_Pitch1.27mm, symbol lmarv:74HC590
- removed U11, U15, U16, U20, U24, U36, U40: IS61LV256AL, lmarv:TSOP-I-28_18.4x8mm_Pitch0.55mm, symbol lmarv:IS61LV256AL
- removed U14, U27, U29, U30, U31, U33, U34, U35, U38, U47, U48, U49, U50, U51, U52, U53, U54, U55: 74LVC541, Housings_SSOP:TSSOP-20_4.4x6.5mm_Pitch0.65mm, symbol lmarv:74LVC541
- removed U2: AT28BV64B-20JU, Sockets:PLCC32, symbol lmarv:AT28BV64B-20JU
- removed U3: AT28BV256B-20JU, Sockets:PLCC32, symbol lmarv:AT28BV256B-20JU
- removed unit 1 of U42
- removed unit 5 of U42
- removed unit 2 of U43
- removed unit 1 of U43
- removed unit 4 of U44
- removed unit 1 of U44
- removed unit 2 of U44
- removed unit 3 of U44
- added P1: dual-pcie-cardedge_split, symbol lmarv:dual-pcie-cardedge_split
- added U1, U11, U15, U16, U20, U24, U36, U40, U42, U43, U44, U57, U58, U59: 74LVC541, Housings_SSOP:TSSOP-20_4.4x6.5mm_Pitch0.65mm, symbol lmarv:74LVC541
- added U14, U35: AT28BV64B-20JU, Sockets:PLCC32, symbol lmarv:AT28BV64B-20JU
- added unit 1 of U2
- added unit 2 of U2
- added U27, U29, U30, U31, U33, U38, U47, U48, U49, U50, U51, U52, U53, U54: IS61LV256AL, lmarv:TSOP-I-28_18.4x8mm_Pitch0.55mm, symbol lmarv:IS61LV256AL
- added U3: 74HC590, Housings_SOIC:SOIC-16_3.9x9.9mm_Pitch1.27mm, symbol lmarv:74HC590
- added U34: AT28BV256B-20JU, Sockets:PLCC32, symbol lmarv:AT28BV256B-20JU
- added unit 1 of U55
- renumbered C19 to C1, C4 to C10, C3 to C11, C2 to C12, C1 to C13, C27 to C14, C26 to C15, C25 to C16, C23 to C17, C22 to C18, C21 to C19, C18 to C2, C10 to C20, C9 to C21, C8 to C22, C20 to C23, C16 to C24, C15 to C25, C11 to C26, C39 to C27, C38 to C28, C37 to C29, C17 to C3, C35 to C30, C34 to C31, C33 to C32, C31 to C33, C30 to C34, C29 to C35, C32 to C37, C28 to C38, C24 to C39, C14 to C4, C50 to C40, C49 to C41, C48 to C42, C47 to C43, C46 to C44, C44 to C46, C43 to C47, C42 to C48, C41 to C49, C13 to C5, C40 to C50, C56 to C51, C55 to C52, C54 to C53, C53 to C54, C52 to C55, C51 to C56, C102 to C57, C101 to C58, C100 to C59, C12 to C6, C6 to C8, C5 to C9, U43 to U2, U44 to U55, U42 to U55
Connections:
- net labels added: CLU_D0, CLU_D1, CLU_D2, CLU_D3, CLU_D4, CLU_D5, CLU_D6, CLU_D7, SLICE1_G, SLICE1_P, SLICE2_D[0], SLICE2_D[1], SLICE2_D[2], SLICE2_D[3], SLICE2_D[4], cin_cla, ~BOOT_WR'
- net labels removed: CLA_D0, CLA_D1, CLA_D2, CLA_D3, CLA_D4, CLA_D5, CLA_D6, CLA_D7, GND, SLICE_D0, SLICE_D1, SLICE_D2, SLICE_D3, SLICE_D4, SLICE_D5, SLICE_D6, SLICE_D7, SW_VCC1, SW_VCC2, SW_VCC3, VDD, cout[0], cout[1], cout[2], cout[3], cout[4], cout[5], cout[6], cout[7], g[7], p[7], ~BOOT_ALU_WR', ~BOOT_CLA_WR
- wire segments 1643 -> 1490
- no-connect marks 60 -> 165
Other:
- note added: "ALU BOOT COUNTER"
- note added: "ARITHMETIC\nBIT SLICE"
- note added: "ARITHMETIC\nBIT SLICE ROM"
- note added: "BUFFER ENABLED DURING\nBOOT PHASE 0"
- note added: "BUFFER ENABLED DURING\nBOOT PHASE 1"
- note added: "BUFFERS ENABLED DURING\nBOOT PHASE 0"
- note added: "BUFFERS ENABLED DURING\nBOOT PHASE 1"
- note added: "CARRY LOOKAHEAD UNIT"
- note added: "CARRY LOOKAHEAD UNIT ROM"
- note added: "PROPAGATE/GENERATE ROM"
- note added: "PROPAGATE/GENERATE\nBIT SLICE"
- note removed: "32k x 8 CARRY\nLOOKAHEAD UNIT"
- note removed: "32k x 8 CLU ROM"
- note removed: "8k x 8 SLICE 0"
- note removed: "8k x 8 SLICE 1"
- note removed: "8k x 8 SLICE 2"
- note removed: "8k x 8 SLICE 3"
- note removed: "8k x 8 SLICE 4"
- note removed: "8k x 8 SLICE 5"
- note removed: "8k x 8 SLICE 6"
- note removed: "8k x 8 SLICE 7"
- note removed: "8k x 8 SLICE ROM"
- note removed: "BOOT LOADER COUNTER"
- moved on the sheet: C1, C10, C11, C12, C13, C14, C15, C16, C17, C18, C19, C2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

Commit message: Update alu.py, add some instruction diagrams
Parts:
- removed U10, U11, U12, U23, U24, U25, U37, U43, U44, U45, U5, U6, U7, U8, U9: 74LVC541, Housings_SSOP:TSSOP-20_4.4x6.5mm_Pitch0.65mm, symbol lmarv:74LVC541
- added U10, U11, U12, U13, U24, U25, U38, U6, U7, U8, U9: 74LVC541_a, Housings_SSOP:TSSOP-20_4.4x6.5mm_Pitch0.65mm, symbol lmarv:74LVC541_a
- added U27: 74LVC541, Housings_SSOP:TSSOP-20_4.4x6.5mm_Pitch0.65mm, symbol lmarv:74LVC541
- C1, C10, C11, C12, C13, C14, C15, C16, C17, C18, C19, C2, C20, C21, C22, C23, C24, C25, C26, C27, C28, C29, C3, C30, C31, C32, C33, C34, C35, C36, C37, C38, C39, C4, C40, C41, C42, C43, C44, C45, C46, C47, C48, C49, C5, C50, C51, C52, C53, C54, C55, C56, C6, C7, C8, C9: value 0u1 -> 100n
- P1: footprint (none) -> lmarv:PCI-EXPRESS
- renumbered U13 to U14, U14 to U15, U15 to U16, U16 to U17, U17 to U18, U18 to U19, U19 to U20, U20 to U21, U21 to U22, U22 to U23, U27 to U28, U28 to U29, U55 to U3, U29 to U30, U30 to U31, U31 to U32, U32 to U33, U33 to U34, U34 to U35, U35 to U36, U36 to U37, U38 to U39, U3 to U4, U39 to U40, U40 to U41, U41 to U42, U42 to U43, U46 to U44, U47 to U45, U48 to U46, U49 to U47, U50 to U48, U51 to U49, U4 to U5, U52 to U50, U53 to U51, U54 to U52, U56 to U53, U57 to U54, U58 to U55, U59 to U56
Connections:
- net labels added: SLICE1_CIN, cmp[7]
- net labels removed: cin_cla, lt[0], lt[1], lt[2], lt[3], lt[4], lt[5], lt[6], lt[7]
- wire segments 1490 -> 1430
- no-connect marks 165 -> 152
Other:
- moved on the sheet: U44

Commit message: ALU rev D, with simulations
Parts:
- removed C10, C11, C12, C13, C17, C18, C19, C20, C21, C23, C24, C53, C54, C55, C56, C6, C7, C8, C9: 100n, Capacitors_SMD:C_0603, symbol Device:C
- removed J1: Conn_02x03_Odd_Even, Connectors_Samtec:SDL-106-X-XX_2x03, symbol Connector_Generic:Conn_02x03_Odd_Even
- removed U10, U11, U12, U13, U6, U7, U8, U9: 74LVC541_a, Housings_SSOP:TSSOP-20_4.4x6.5mm_Pitch0.65mm, symbol lmarv:74LVC541_a
- removed U17, U18, U19, U20, U21, U22, U23, U53, U54, U55, U56: 74LVC541, Housings_SSOP:TSSOP-20_4.4x6.5mm_Pitch0.65mm, symbol lmarv:74LVC541
- removed U4, U5: 74HC590, Housings_SOIC:SOIC-16_3.9x9.9mm_Pitch1.27mm, symbol lmarv:74HC590
- added C57, C58, C59: 100n, Capacitor_SMD:C_0603_1608Metric, symbol Device:C
- added D1, D2: APTD2012LSURCK, lmarv:D_0805_Wide, symbol Device:LED_ALT
- added R4: 10k, Resistor_SMD:R_0603_1608Metric, symbol Device:R
- added R5, R6: 3k3, Resistor_SMD:R_0603_1608Metric, symbol Device:R
- added U59: 74LS157, Package_SO:TSSOP-16_4.4x5mm_P0.65mm, symbol Logic_74xx:74LS157
- C1, C14, C15, C16, C2, C25, C26, C27, C28, C29, C3, C30, C31, C32, C33, C34, C35, C36, C37, C38, C39, C4, C40, C41, C42, C43, C44, C45, C46, C47, C48, C49, C5, C50, C51, C52: footprint Capacitors_SMD:C_0603 -> Capacitor_SMD:C_0603_1608Metric
- C100: renamed from C59; footprint Capacitors_SMD:CP_Elec_4x4.5 -> Capacitor_SMD:CP_Elec_4x4.5
- C101: renamed from C58; footprint Capacitors_SMD:CP_Elec_4x4.5 -> Capacitor_SMD:CP_Elec_4x4.5
- C102: renamed from C57; footprint Capacitors_SMD:CP_Elec_4x4.5 -> Capacitor_SMD:CP_Elec_4x4.5
- C24: renamed from C22; footprint Capacitors_SMD:C_0603 -> Capacitor_SMD:C_0603_1608Metric
- R1, R2, R3: footprint Resistors_SMD:R_0603 -> Resistor_SMD:R_0603_1608Metric
- U1, U14, U16, U24, U25, U26, U27, U37, U38, U40, U41, U42, U43, U44: footprint Housings_SSOP:TSSOP-20_4.4x6.5mm_Pitch0.65mm -> Package_SO:TSSOP-20_4.4x6.5mm_P0.65mm
- U15: footprint Sockets:PLCC32 -> Package_LCC:PLCC-32_THT-Socket
- U2, U3: footprint Housings_SSOP:TSSOP-14_4.4x5mm_Pitch0.65mm -> Package_SO:TSSOP-14_4.4x5mm_P0.65mm
Connections:
- net labels added: cin0', cin0_boot, ~BOOT_PH0_WR, ~BOOT_PH1_WR, ~alu_oe_led
- net labels removed: ~BOOT_RCO
- wire segments 1430 -> 1341
- no-connect marks 152 -> 151
Other:
- note added: "A15&~ALU_BOOT_WR~"
- moved on the sheet: P1A, P1B, P1C, P1D, R1, R2, U1, U2A, U3B, U3C, U3D
