File: lmarv-1/ram-based-register-card/ram-based-register-card.sch (KiCad schematic (older format))
At the start: 17 parts, among them P1 dual-pcie-cardedge, U1 IDT70V24_TQ100, U2 IDT70V24_TQ100, U3 IDT70V24_TQ100, U4 IDT70V24_TQ100

Commit message: ALU rev D, with simulations
Parts:
- removed P1: dual-pcie-cardedge, lmarv:PCI-EXPRESS, symbol lmarv:dual-pcie-cardedge
- added C37, C38, C39: 0u1, Capacitor_SMD:C_0603_1608Metric, symbol Device:C
- added P1: dual-pcie-cardedge_split, lmarv:PCI-EXPRESS, symbol lmarv:dual-pcie-cardedge_split
- added R1, R2, R3, R4, R5: 47k, Resistor_SMD:R_0603_1608Metric, symbol Device:R
- added U21, U22: 74LVC138, Package_SO:TSSOP-16_4.4x5mm_P0.65mm, symbol Logic_74xx:74LS138
- added U23: 74LVC04, Package_SO:TSSOP-14_4.4x5mm_P0.65mm, symbol Logic_74xx:74LS04
- C1, C10, C11, C12, C2, C3, C4, C5, C6, C7, C8, C9: footprint Capacitors_SMD:C_0603 -> Capacitor_SMD:C_0603_1608Metric
- U1, U2, U3, U4: footprint Housings_QFP:TQFP-100_14x14mm_Pitch0.5mm -> Package_QFP:TQFP-100_14x14mm_P0.5mm
Connections:
- net labels added: rd[0]', rd[10]', rd[11]', rd[12]', rd[13]', rd[14]', rd[15]', rd[16]', rd[17]', rd[18]', rd[19]', rd[1]', rd[20]', rd[21]', rd[22]', rd[23]', rd[24]', rd[25]', rd[26]', rd[27]', rd[28]', rd[29]', rd[2]', rd[30]', rd[31]', rd[3]', rd[4]', rd[5]', rd[6]', rd[7]', rd[8]', rd[9]', rda[0]', rda[1]', rda[2]', rda[3]', rda[4]', rs1[0]', rs1[10]', rs1[11]', rs1[12]', rs1[13]', rs1[14]', rs1[15]', rs1[16]', rs1[17]', rs1[18]', rs1[19]', rs1[1]', rs1[20]', rs1[21]', rs1[22]', rs1[23]', rs1[24]', rs1[25]', rs1[26]', rs1[27]', rs1[28]', rs1[29]', rs1[2]', rs1[30]', rs1[31]', rs1[3]', rs1[4]', rs1[5]', rs1[6]', rs1[7]', rs1[8]', rs1[9]', rs1_zero, rs1a[0]', rs1a[1]', rs1a[2]', rs1a[3]', rs1a[4]', rs2[0]', rs2[10]', rs2[11]', rs2[12]', rs2[13]', rs2[14]', rs2[15]', rs2[16]', rs2[17]', rs2[18]', rs2[19]', rs2[1]', rs2[20]', rs2[21]', rs2[22]', rs2[23]', rs2[24]', rs2[25]', rs2[26]', rs2[27]', rs2[28]', rs2[29]', rs2[2]', rs2[30]', rs2[31]', rs2[3]', rs2[4]', rs2[5]', rs2[6]', rs2[7]', rs2[8]', rs2[9]', rs2_zero, rs2a[0]', rs2a[1]', rs2a[2]', rs2a[3]', rs2a[4]', ~rd_wr~', ~rs1_rd~', ~rs1_zero, ~rs2_rd~', ~rs2_zero
- net labels removed: ~rd_bhh, ~rd_bhl, ~rd_blh, ~rd_bll, ~rs1_bhh, ~rs1_bhl, ~rs1_blh, ~rs1_bll, ~rs2_bhh, ~rs2_bhl, ~rs2_blh, ~rs2_bll
- wire segments 550 -> 1029
- no-connect marks 8 -> 70
Other:
- note removed: "DATA LINES ARE REVERSED ON PURPOSE.\nTHIS IS WHY ~UB~ AND ~LB~ ARE ALSO REVERSED."
- note removed: "HIGH HALF"
- note removed: "LOW HALF"
- note removed: "RD = DATA, DESTINATION REGISTER\nRDA = ADDRESS, DESTINATION REGISTER\nRS1 = DATA, SOURCE REGISTER 1\nRS1A = ADDRESS, SOURCE REGISTER 1\nRS2 = DATA, SOURCE REGISTER 2\nRS2A = ADDRESS, SOURCE REGISTER 2"
- note removed: "~RD_WR~ = WRITE DESTINATION REGISTER\n~RD_BHH~ = DESTINATION REGISTER BYTE 3\n~RD_BHL~ = DESTINATION REGISTER BYTE 2\n~RD_BLH~ = DESTINATION REGISTER BYTE 1\n~RD_BLL~ = DESTINATION REGISTER BYTE 0\n\n~RS1_RD~ = READ SOURCE REGISTER 1\n~RS1_BHH~ = SOURCE REGISTER 1 BYTE 3\n~RS1_BHL~ = SOURCE REGISTER 1 BYTE 2\n~RS1_BLH~ = SOURCE REGISTER 1 BYTE 1\n~RS1_BLL~ = SOURCE REGISTER 1 BYTE 0\n\n~RS2_RD~ =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"
- moved on the sheet: C1, C10, C11, C12, C2, C3, C4, C5, C6, C7, C8, C9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
